File: BirthdayBuzzer.kicad_sch (KiCad schematic)
At the start: 14 parts, among them J3 Conn_ARM_SWD_TagConnect_TC203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, SW1 SW_Push, U1 PIC18F15Q41-I/SS

Commit message: Cleaned up schematics and added notes
Connections:
- no-connect marks 0 -> 8
Other:
- title: (none) -> BirthdayBuzzer
- moved on the sheet: BT1, BZ1, C1, J3, SW1, U1

Commit message: Fixed Capacitor in Schematics and GND in layout
Parts:
- C1: value C -> 10uF
Connections:
- net GND: now also C1.1
- net +3V6: now reaches C1.2, U1.1 (VDD)
- net +3V6: now also BT1.1 (+), D1.4 (A), D2.4 (A), J3.1 (VCC)
- removed net +3V0: BT1.1 (+), C1.1, D1.4 (A), D2.4 (A), J3.1 (VCC)
Other:
- moved on the sheet: C1
Changed lines of the file:
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@@
 		(comment 1 "Author: Christian R")
+	)
+	(junction
+		(at 57.15 60.96)
+		(diameter 0)
+		(color 0 0 0 0)
 	)
 	(no_connect
@@
 	(wire
 		(pts
-			(xy 57.15 58.42) (xy 57.15 59.69)
+			(xy 57.15 58.42) (xy 57.15 60.96)
 		)
 		(stroke
@@
 	(wire
 		(pts
+			(xy 49.53 60.96) (xy 49.53 62.23)
+		)
+		(stroke
+			(width 0)
+			(type default)
+		)
+	)
+	(wire
+		(pts
 			(xy 133.35 59.69) (xy 138.43 59.69)
 		)
@@
 		(pts
 			(xy 24.13 139.7) (xy 24.13 144.78)
+		)
+		(stroke
+			(width 0)
+			(type default)
+		)
+	)
+	(wire
+		(pts
+			(xy 57.15 60.96) (xy 57.15 67.31)
 		)
 		(stroke
@@
 	(symbol
 		(lib_id "Device:C")
-		(at 57.15 63.5 0)
+		(at 53.34 60.96 90)
 		(unit 1)
 		(exclude_from_sim no)
@@
 		(on_board yes)
 		(dnp no)
-		(fields_autoplaced yes)
 		(property "Reference" "C1"
-			(at 60.96 62.2299 0)
-			(effects
-				(font
-					(size 1.27 1.27)
-				)
-				(justify left)
-			)
-		)
-		(property "Value" "C"
-			(at 60.96 64.7699 0)
-			(effects
-				(font
-					(size 1.27 1.27)
-				)
-				(justify left)
+			(at 49.276 55.372 90)
+			(effects
+				(font
+					(size 1.27 1.27)
+				)
+			)
+		)
+		(property "Value" "10uF"
+			(at 49.276 57.912 90)
+			(effects
+				(font
+					(size 1.27 1.27)
+				)
 			)
 		)
 		(property "Footprint" "Capacitor_THT:C_Disc_D4.3mm_W1.9mm_P5.00mm"
-			(at 58.1152 67.31 0)
+			(at 57.15 59.9948 0)
 			(effects
 				(font
@@
 		)
 		(property "Datasheet" "~"
-			(at 57.15 63.5 0)
+			(at 53.34 60.96 0)
 			(effects
 				(font
@@
 		)
 		(property "Description" "Unpolarized capacitor"
-			(at 57.15 63.5 0)
+			(at 53.34 60.96 0)
 			(effects
 				(font
@@
 			)
 		)
-		(property "Value" "+3V0"
+		(property "Value" "+3V6"
 			(at 22.352 135.382 0)
 			(effects
@@
 			)
 		)
-		(property "Value" "+3V0"
+		(property "Value" "+3V6"
 			(at 216.662 64.262 0)
 			(effects
@@
 				(path "/9c0e249a-475f-406b-99f3-8e689c92e153"
 					(reference "BT1")
+					(unit 1)
+				)
+			)
+		)
+	)
+	(symbol
+		(lib_id "power:GND")
+		(at 49.53 62.23 0)
+		(unit 1)
+		(exclude_from_sim no)
+		(in_bom yes)
+		(on_board yes)
+		(dnp no)
+		(property "Reference" "#PWR011"
+			(at 49.53 68.58 0)
+			(effects
+				(font
+					(size 1.27 1.27)
+				)
+				(hide yes)
+			)
+		)
+		(property "Value" "GND"
+			(at 49.784 66.04 0)
+			(effects
+				(font
+					(size 1.27 1.27)
+				)
+			)
+		)
+		(property "Footprint" ""
+			(at 49.53 62.23 0)
+			(effects
+				(font
+					(size 1.27 1.27)
+				)
+				(hide yes)
+			)
+		)
+		(property "Datasheet" ""
+			(at 49.53 62.23 0)
+			(effects
+				(font
+					(size 1.27 1.27)
+				)
+				(hide yes)
+			)
+		)
+		(property "Description" "Power symbol creates a global label with name \"GND\" , ground"
+			(at 49.53 62.23 0)
+			(effects
+				(font
+					(size 1.27 1.27)
+				)
+				(hide yes)
+			)
+		)
+		(pin "1"
+		)
+		(instances
+			(project "BirthdayBuzzer"
+				(path "/9c0e249a-475f-406b-99f3-8e689c92e153"
+					(reference "#PWR011")
 					(unit 1)
 				)
@@
 			)
 		)
-		(property "Value" "+3V0"
+		(property "Value" "+3V6"
 			(at 22.352 165.862 0)
 			(effects
@@
 			)
 		)
-		(property "Value" "+3V0"
+		(property "Value" "+3V6"
 			(at 83.312 23.622 0)
 			(effects
@@
 			)
 		)
-		(property "Value" "+3V0"
+		(property "Value" "+3V6"
 			(at 55.372 54.102 0)
 			(effects
